File: CY7CBreakout.kicad_pcb (KiCad board)
At the start: 2 copper layers, 52 x 27.9 mm, 36 parts, among them J1 PORTA, J2 PORTB, J3 PORTD, J4 POWER, J5 WP, J6 +5V Source, U1 CY7C68013A-56LTX, U2 M24128, U3 TLV755P, Y1 24MHz

Commit message: Added the OSHW logo to the silkscreen for the board
Parts:
- added LOGO1: Logo_Open_Hardware_Small, Symbol:OSHW-Logo2_7.3x6mm_SilkScreen, F.Cu at (123.5, 96.7)
